File: hardware/carrier/usb_serial.kicad_sch (KiCad schematic)
At the start: 17 parts, among them Q2 UMH3N, U5 CP2102N-A02-GQFN24, U6 SN74LVC2G126DCUR

Commit message: hardware/carrier: front light is the GDEY029T94-FL03 (6-pin flex -> FH34SRJ-6S on the panel board, anode/cathode over a 10-way SH cable, 33R 1206 + Q4 PWM drive replaces the NSI45020), front-light button SW2 on IO4 (FL_BTN), low-profile pass (FH34SRJ 1.0 mm ZIFs, 2 x 100uF 0805 instead of the 2.5 mm 1210, part-height table), sleep-current audit (Q1 gate pull-up 100k -> 2.2M: 38 -> 1.9 uA; SN74LVC2G126 moved to the bus-powered BRG_VDD rail: 0 on battery; table in the README), TPS62840 has no fixed-3.3 V variant (README). Custom FH34SRJ footprints from the Hirose catalog; LCSC numbers via the JLCPCB parts API. Both boards re-placed and re-routed: 0 unconnected, 0 clearance/courtyard errors, silk notes only; ERC 0/0; exports refreshed (owner, 17 Oct 2026)
Co-Authored-By: Claude Fable 5.1 <noreply@anthropic.com>
Parts:
- removed C14: 4.7uF, Capacitor_SMD:C_0603_1608Metric, symbol Device:C
- added C19: 100nF, Capacitor_SMD:C_0603_1608Metric, symbol Device:C
- C15, C17: value 100nF -> 4.7uF; LCSC C14663 -> C19666; MPN CL10B104KB8NNNC -> CL10A475KP8NNNC
- C16: value 4.7uF -> 100nF; LCSC C19666 -> C14663; MPN CL10A475KP8NNNC -> CL10B104KB8NNNC
Connections:
- net 3V3: no longer C18.1, U6.8 (VCC)
- net BRG_VDD: now also C18.1, U6.8 (VCC), C19.1; no longer C16.1
- net GND: now also C19.2
- net VBUS: now also C16.1
Other:
- note added: "U6 SN74LVC2G126: both OE from VBUS_DET. A: ESP_TX0 -> BRG_RXD. B: BRG_TXD -> ESP_RX0. 10k keeps ESP_RX0 high with no cable. U6 VCC is BRG_VDD (bus-powered): with no cable the buffer is unpowered (Ioff outputs), so no LVC quiescent/float current on the battery."
- note removed: "U6 SN74LVC2G126: both OE from VBUS_DET. A: ESP_TX0 -> BRG_RXD. B: BRG_TXD -> ESP_RX0. 10k keeps ESP_RX0 high with no cable."
- moved on the sheet: C15, C16, C17, C18
