File: hardware/carrier/usb_serial.kicad_sch (KiCad schematic)
At the start: 17 parts, among them Q2 UMH3N, U5 CP2102N-A02-GQFN24, U6 SN74LVC2G126DCUR

Commit message: Manually review and fix carrier board schematic
The initial product of clause was mostly okay electrically
but impossible to read. This is a fully redone version
that has all circuits reverified with some modifications.
Connections:
- net BRG_DTR: now also R25.1; no longer R24.1
- net BRG_RTS: now also R24.1; no longer R25.1
- net GND: now also C17.1, C18.1; no longer C17.2, C18.2
- net BRG_RST: no longer names the net of R21.1, U5.9 (~{RST})
- net BRG_VBUS_SNS: no longer names the net of R22.2, R23.1, U5.8 (VBUS)
- net BRG_VDD: no longer names the net of C19.1, R21.2, U5.5 (VIO), U5.6 (VDD), U6.8 (VCC)
- net BRG_VDD: now also C17.2, C18.2; no longer C17.1, C18.1
Other:
- note added: "U6 SN74LVC2G126: both OE from VBUS_DET. A: ESP_TX0 -> BRG_RXD. B: BRG_TXD -> ESP_RX0. 10k keeps ESP_RX0 high with no cable. U6 VCC is BRG_3V3 (bus-powered): with no cable the buffer is unpowered (Ioff outputs), so no LVC quiescent/float current on the battery."
- note added: "USB-serial bridge: bus-powered CP2102N (unpowered without a cable) SN74LVC2G126 isolates UART0 when VBUS_DET is low Espressif two-transistor auto-reset."
- note removed: "U6 SN74LVC2G126: both OE from VBUS_DET. A: ESP_TX0 -> BRG_RXD. B: BRG_TXD -> ESP_RX0. 10k keeps ESP_RX0 high with no cable. U6 VCC is BRG_VDD (bus-powered): with no cable the buffer is unpowered (Ioff outputs), so no LVC quiescent/float current on the battery."
- note removed: "USB-serial bridge: bus-powered CP2102N (unpowered without a cable), SN74LVC2G126 isolates UART0 when VBUS_DET is low, Espressif two-transistor auto-reset."
- moved on the sheet: C15, C16, C17, C18, C19, JP1, Q2A, Q2B, R21, R22, R23, R24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
