File: hardware/carrier/peripherals.kicad_sch (KiCad schematic)
At the start: 26 parts, among them J4 CARDKB, J6 MSG_LED, J7 HAPTIC, Q4 2N7002, SW2 SKQGAFE010, U7 LIS2DW12TR, U9 DRV2605LDGSR

Commit message: Manually review and fix carrier board schematic
The initial product of clause was mostly okay electrically
but impossible to read. This is a fully redone version
that has all circuits reverified with some modifications.
Parts:
- removed C21, C24, C26: 100nF, Capacitor_SMD:C_0603_1608Metric, symbol Device:C
- removed C22, C23: 10uF, Capacitor_SMD:C_0603_1608Metric, symbol Device:C
- removed C25, C27: 1uF, Capacitor_SMD:C_0603_1608Metric, symbol Device:C
- removed D5: RED, LED_SMD:LED_0603_1608Metric, symbol Device:LED
- removed J4: CARDKB, Connector_JST:JST_PH_S4B-PH-SM4-TB_1x04-1MP_P2.00mm_Horizontal, symbol Connector_Generic:Conn_01x04
- removed J6: MSG_LED, Connector_JST:JST_SH_SM02B-SRSS-TB_1x02-1MP_P1.00mm_Horizontal, symbol Connector_Generic:Conn_01x02
- removed J7: HAPTIC, Connector_JST:JST_SH_SM02B-SRSS-TB_1x02-1MP_P1.00mm_Horizontal, symbol Connector_Generic:Conn_01x02
- removed Q4: 2N7002, Package_TO_SOT_SMD:SOT-23, symbol Transistor_FET:2N7002
- removed R29, R30, R31, R32: 4.7k, Resistor_SMD:R_0603_1608Metric, symbol Device:R
- removed R33: 33R, Resistor_SMD:R_1206_3216Metric, symbol Device:R
- removed R34: 100R, Resistor_SMD:R_0603_1608Metric, symbol Device:R
- removed R35, R36, R39: 100k, Resistor_SMD:R_0603_1608Metric, symbol Device:R
- removed R37: 330R, Resistor_SMD:R_0603_1608Metric, symbol Device:R
- removed R38: 1k, Resistor_SMD:R_0603_1608Metric, symbol Device:R
- removed SW2: SKQGAFE010, Button_Switch_SMD:SW_SPST_SKQG_WithoutStem, symbol Switch:SW_Push
- removed U7: LIS2DW12TR, Package_LGA:LGA-12_2x2mm_P0.5mm, symbol pager-carrier:LIS2DW12TR
- removed U9: DRV2605LDGSR, Package_SO:TSSOP-10_3x3mm_P0.5mm, symbol pager-carrier:DRV2605LDGSR
Connections:
- no-connect marks 2 -> 0
Other:
- note removed: "Front light GDEY029T94-FL03: 4 white LEDs in parallel on its own 6-pin 0.5 mm flex (1-2 anode, 3-4 NC, 5-6 cathode), Vf 2.75-3.3 V, 60 mA max. The 6-pin ZIF sits on the panel board; anode/cathode ride the panel cable (J3 pins 9/10). R-FL 33R from SYS_SW sets 18 mA at a 3.4 V cell, 42 mA at 4.2 V, 50 mA on USB (SYS 4.45 V). Q4 low-side switch, PWM from FL_PWM (IO7) for dimming / battery compensati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"
- note removed: "Haptic (DNP): DRV2605L on I2C1 (0x5A), EN = HAPTIC_EN (IO6) with 100k pull-down, IN/TRIG to GND (I2C trigger), OUT+/- to J7."
- note removed: "J4 CardKB (Grove order): 1 KBD_SCL, 2 KBD_SDA, 3 3V3_OUT, 4 GND. Pull-ups to 3V3_OUT so they vanish with the rail."
- note removed: "Place U7 away from J7 and the panel cable; X axis along the tin's long edge; mark orientation on silk."
- note removed: "SW2 front-light button: FL_BTN (IO4, RTC GPIO, ext1 wake-capable) to GND, 100k pull-up to the always-on 3V3, 100nF debounce. No current while idle."
- note removed: "U7 LIS2DW12 on I2C1 (ACC_*), SA0 low = 0x18, CS high = I2C mode, INT1 -> IO16 (RTC wake). Always on from 3V3."
