File: hardware/carrier/power.kicad_sch (KiCad schematic)
At the start: 42 parts, among them J1 USB4235, J2 BATTERY, Q1 DMG2305UX-7, SW1 JS102011SAQN, U1 BQ25185DLHR, U10 MAX17048G+T10, U3 TPS62840DLCR, U4 TPS22917DBV

Commit message: Manually review and fix carrier board schematic
The initial product of clause was mostly okay electrically
but impossible to read. This is a fully redone version
that has all circuits reverified with some modifications.
Parts:
- removed C10: 1uF, Capacitor_SMD:C_0603_1608Metric, symbol Device:C
- removed C2: 10uF/25V, Capacitor_SMD:C_0805_2012Metric, symbol Device:C
- removed C9: 1nF, Capacitor_SMD:C_0603_1608Metric, symbol Device:C
- removed F1: 2A PTC, Fuse:Fuse_1206_3216Metric, symbol Device:Polyfuse
- removed R10: 13k, Resistor_SMD:R_0603_1608Metric, symbol Device:R
- removed R20, R6, R7: 0R, Resistor_SMD:R_0603_1608Metric, symbol Device:R
- removed U4: TPS22917DBV, Package_TO_SOT_SMD:SOT-23-6, symbol Power_Management:TPS22917DBV
- added TP1: GND, TestPoint:TestPoint_Pad_1.0x1.0mm, symbol Connector:TestPoint
- added TP2: VBUS, TestPoint:TestPoint_Pad_1.0x1.0mm, symbol Connector:TestPoint
- added TP3: SYS, TestPoint:TestPoint_Pad_1.0x1.0mm, symbol Connector:TestPoint
- added TP4: SYS_SW, TestPoint:TestPoint_Pad_1.0x1.0mm, symbol Connector:TestPoint
- added TP5: VBAT, TestPoint:TestPoint_Pad_1.0x1.0mm, symbol Connector:TestPoint
- added TP6: 3V3, TestPoint:TestPoint_Pad_1.0x1.0mm, symbol Connector:TestPoint
- C4: value 22uF -> 10uF; footprint Capacitor_SMD:C_0805_2012Metric -> Capacitor_SMD:C_0603_1608Metric; LCSC C45783 -> C19702; MPN CL21A226MAQNNNE -> CL10A106KP8NNNC
- Q1: value DMG2305UX-7 -> AO3401A
Connections:
- net BAT_CELL is gone; now on net VBAT: J2.1 (Pin_1)
- net CHG_CE is gone; now on net GND: U1.4 (~{CE})
- net 3V3: now also R12.1, R13.1, TP6.1; no longer R12.2, R13.2, R18.2
- net CHG_STAT1: now also R12.2; no longer R12.1
- net CHG_STAT2: now also R13.2; no longer R13.1
- net GND: now also TP1.1
- net SYS: now also TP3.1
- net SYS_SW: now also R18.1, TP4.1
- net USB_DM: now also D4.6 (I/O1); no longer D4.3 (I/O2), D4.4 (I/O2), J1.A7 (D-), J1.B7 (D-)
- net USB_DP: now also D4.4 (I/O2); no longer D4.1 (I/O1), D4.6 (I/O1), J1.A6 (D+), J1.B6 (D+)
- net VBAT: now also TP5.1
- net VBUS: now also TP2.1
- net ACC_SCL renamed AON_SCL
- net ACC_SDA renamed AON_SDA
- net BUCK_EN: no longer names the net of R16.2, U3.4 (EN)
- net BUCK_MODE: no longer names the net of R17.1, U3.3 (MODE)
- net BUCK_MODE: now also R18.2; no longer R18.1
- net BUCK_SW: no longer names the net of L2.1, U3.7 (SW)
- net BUCK_VSET: no longer names the net of R19.1, U3.5 (VSET)
- net CHG_ILIM: no longer names the net of R9.1, U1.7 (ILIM/VSET)
- net CHG_IN: no longer names the net of C3.1, R5.2, U1.10 (IN)
- net CHG_ISET: no longer names the net of R11.1, U1.8 (ISET)
- net CHG_TS: no longer names the net of R8.1, U1.6 (TS/MR)
- net PWR_GATE: no longer names the net of C6.1, Q1.1 (G), R14.2, R15.1
- net SW_COM: no longer names the net of R14.1, SW1.2 (B)
- net USB_CC1: no longer names the net of J1.A5 (CC1)
- net USB_CC1: now also R2.1; no longer R1.1
- net USB_CC2: no longer names the net of J1.B5 (CC2)
- net USB_CC2: now also R1.1; no longer R2.1
- new net: D4.3 (I/O2), J1.A6 (D+), J1.B6 (D+)
- new net: D4.1 (I/O1), J1.A7 (D-), J1.B7 (D-)
- no-connect marks 4 -> 3
Other:
- note added: "3.3 V always-on rail: TPS62840DLCR buck from SYS_SW, 2.2uH, 10uF in/out. VSET 267k = 3.3 V. MODE low = power-save (DNP 0R to 3V3 can force PWM)"
- note added: "Battery + Fuel Gauge Battery: J2 (pin 1 = +) Fuel gauge U10 MAX17048. Before the switch to track while off, ~3 uA I2C1 (ACC_*), addr 0x36. QSTRT and CTG low."
- note added: "Charger BQ25185DLHR: ISET 604R = 497 mA fast charge. ILIM/VSET 18k = 500 mA input limit, 4.20 V (13k DNP = 1.1 A). TS unused: 10k to GND."
- note added: "Charger and on/off switch. Switch: SW1 drives only the Q1 gate. Base = GND = ON. 2.2M gate pull-up = off when floating (1.9 uA through the ON switch) 10k + 22nF soft-start limits inrush into the Walter bulk caps."
- note added: "D4: flow-through TVS for ESD protection. Connector pads into pins 1/3, out of pins 6/4 toward U5."
- note added: "Test Points"
- note added: "VBUS detect; enabls U6. 56k/100k divider for 5V -> 3.2V level conversion"
- note removed: "3.3 V always-on rail: TPS62840DLCR buck from SYS_SW, 2.2uH, 10uF in/out. EN from SYS_SW via 100k. VSET 267k = 3.3 V. MODE low = power-save (DNP 0R to 3V3 tries forced PWM if the e-ink shows ripple). STOP low. VOS senses 3V3."
- note removed: "Battery: J2 (pin 1 = +) through F1 2 A PTC to VBAT. Switch: SW1 drives only the Q1 gate; SYS_SW = SYS when on. 2.2M gate pull-up = off when floating (1.9 uA through the ON switch, was 38 uA with 100k); 10k + 22nF soft-start limits inrush into the Walter bulk caps."
- note removed: "Charger BQ25185DLHR: ISET 604R = 497 mA fast charge. ILIM/VSET 18k = 500 mA input limit, 4.20 V (13k DNP = 1.1 A). TS unused: 10k to GND. CE is active-low: 0R to GND. STAT1/2 open-drain, 10k to 3V3."
- note removed: "D4: flow-through TVS. Connector pads into pins 1/3, out of pins 6/4 toward U5."
- note removed: "Display rail: U4 TPS22917 load switch 3V3 -> 3V3_EPD, ON = EPD_ENA (IO12), CT 1nF (~1 ms rise). R-EPD 0R in series to measure panel standby current. QOD open."
- note removed: "Fuel gauge U10 MAX17048 on VBAT (before the switch: keeps tracking while off, ~3 uA). I2C1 (ACC_*), addr 0x36. QSTRT and CTG low."
- note removed: "QOD left open (no quick discharge); tie to VOUT if a fast panel power-down is wanted."
- note removed: "SW1: common (pin 2) -> SW_COM. Pin 1 -> GND = ON. Pin 3 -> SYS = OFF."
- note removed: "SYS is driven by U1 SYS (power output): no PWR_FLAG. 3V3 is only sensed by U3 VOS, so it carries one."
- note removed: "VBUS detect: 56k/100k divider -> VBUS_DET (IO15, 3.2 V at 5 V); also enables U6."
- moved on the sheet: C1, C11, C3, C5, C6, C7, C8, D4, J1, J2, L2, Q1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

Commit message: Fix some small errors and clean up BOM
Parts:
- Q1: LCSC C150470 -> C15127; MPN DMG2305UX-7 -> AO3401A; Note or AO3401A -> or DMG2305UX-7 / C150470
Changed lines of the file:
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@@
 			)
 		)
-		(property "MPN" "DMG2305UX-7"
+		(property "MPN" "AO3401A"
 			(at 80.01 130.81 0)
 			(hide yes)
@@
 			)
 		)
-		(property "LCSC" "C150470"
+		(property "LCSC" "C15127"
 			(at 77.47 130.81 0)
 			(hide yes)
@@
 			)
 		)
-		(property "Note" "or AO3401A"
+		(property "Note" "or DMG2305UX-7 / C150470"
 			(at 72.39 130.81 0)
 			(hide yes)
