File: hardware/carrier/power_components.kicad_sch (KiCad schematic)
At the start: 35 parts, among them J6 USB4235, J7 BATTERY, Q4 AO3401A, SW2 JS102011SAQN, U5 BQ25185DLHR, U6 MAX17048G+T10, U7 TPS62840DLCR

Commit message: Carrier: hand-layout WIP, Walter pins remapped, panel header J1 10 -> 8 pins (owner)
Co-Authored-By: Claude Fable 5.1 <noreply@anthropic.com>
Parts:
- removed TP10: VBAT, TestPoint:TestPoint_Pad_1.0x1.0mm, symbol Connector:TestPoint
- removed TP11: 3V3, TestPoint:TestPoint_Pad_1.0x1.0mm, symbol Connector:TestPoint
- removed TP7: VBUS, TestPoint:TestPoint_Pad_1.0x1.0mm, symbol Connector:TestPoint
- removed TP8: SYS, TestPoint:TestPoint_Pad_1.0x1.0mm, symbol Connector:TestPoint
- removed TP9: SYS_SW, TestPoint:TestPoint_Pad_1.0x1.0mm, symbol Connector:TestPoint
Other:
- note removed: "Test Points"
