File: hardware/carrier/power_components.kicad_sch (KiCad schematic)
At the start: 30 parts, among them J6 USB4235, J7 BATTERY, Q4 AO3401A, SW2 JS102011SAQN, U5 BQ25185DLHR, U6 MAX17048G+T10, U7 TPS62840DLCR

Commit message: Carrier: close the outline, tidy silkscreen, add GND pours (DRC 278 -> 28)
- Edge.Cuts rebuilt as a single closed loop (right edge 113.15, SIM notch, 1 mm corners)
- 0402/LGA parts moved to pager-carrier:*_NoSilk footprints (library copies without the
  silk outline), schematic fields updated; J6 silk box stops short of the shield pads;
  reference text re-placed or hidden; stale board texts removed
- GND pours both layers (0.2 clearance, thermal reliefs), 3 stitching vias for the
  top-side GND groups that had no path to the plane; all GND connected
- Remaining: 4 owner routing clearances, H1-H3 parked off-board, 2 unrouted nets

Co-Authored-By: Claude Fable 5.1 <noreply@anthropic.com>
Parts:
- C14, C15, C16, C17, C18, C19: footprint Capacitor_SMD:C_0402_1005Metric -> pager-carrier:C_0402_1005Metric_NoSilk
- L1: footprint Inductor_SMD:L_Murata_DFE201610P -> pager-carrier:L_Murata_DFE201610P_NoSilk
- R23, R24, R25, R26, R27, R28, R29, R30, R31, R32, R33, R34, R37, R38: footprint Resistor_SMD:R_0402_1005Metric -> pager-carrier:R_0402_1005Metric_NoSilk
Changed lines of the file:
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@@
 			)
 		)
-		(property "Footprint" "Capacitor_SMD:C_0402_1005Metric"
+		(property "Footprint" "pager-carrier:C_0402_1005Metric_NoSilk"
 			(at 82.55 173.99 0)
 			(hide yes)
@@
 			)
 		)
-		(property "Footprint" "Capacitor_SMD:C_0402_1005Metric"
+		(property "Footprint" "pager-carrier:C_0402_1005Metric_NoSilk"
 			(at 154.94 59.69 0)
 			(hide yes)
@@
 			)
 		)
-		(property "Footprint" "Capacitor_SMD:C_0402_1005Metric"
+		(property "Footprint" "pager-carrier:C_0402_1005Metric_NoSilk"
 			(at 78.74 121.92 0)
 			(hide yes)
@@
 			)
 		)
-		(property "Footprint" "Resistor_SMD:R_0402_1005Metric"
+		(property "Footprint" "pager-carrier:R_0402_1005Metric_NoSilk"
 			(at 215.9 76.2 0)
 			(hide yes)
@@
 			)
 		)
-		(property "Footprint" "Resistor_SMD:R_0402_1005Metric"
+		(property "Footprint" "pager-carrier:R_0402_1005Metric_NoSilk"
 			(at 33.02 179.07 0)
 			(hide yes)
@@
 			)
 		)
-		(property "Footprint" "Resistor_SMD:R_0402_1005Metric"
+		(property "Footprint" "pager-carrier:R_0402_1005Metric_NoSilk"
 			(at 72.39 50.8 0)
 			(hide yes)
@@
 			)
 		)
-		(property "Footprint" "Capacitor_SMD:C_0402_1005Metric"
+		(property "Footprint" "pager-carrier:C_0402_1005Metric_NoSilk"
 			(at 135.89 162.56 0)
 			(hide yes)
@@
 			)
 		)
-		(property "Footprint" "Resistor_SMD:R_0402_1005Metric"
+		(property "Footprint" "pager-carrier:R_0402_1005Metric_NoSilk"
 			(at 25.4 179.07 0)
 			(hide yes)
@@
 			)
 		)
-		(property "Footprint" "Resistor_SMD:R_0402_1005Metric"
+		(property "Footprint" "pager-carrier:R_0402_1005Metric_NoSilk"
 			(at 146.05 44.45 0)
 			(hide yes)
@@
 			)
 		)
-		(property "Footprint" "Resistor_SMD:R_0402_1005Metric"
+		(property "Footprint" "pager-carrier:R_0402_1005Metric_NoSilk"
 			(at 85.09 121.92 0)
 			(hide yes)
@@
 			)
 		)
-		(property "Footprint" "Resistor_SMD:R_0402_1005Metric"
+		(property "Footprint" "pager-carrier:R_0402_1005Metric_NoSilk"
 			(at 41.91 129.54 0)
 			(hide yes)
@@
 			)
 		)
-		(property "Footprint" "Resistor_SMD:R_0402_1005Metric"
+		(property "Footprint" "pager-carrier:R_0402_1005Metric_NoSilk"
 			(at 40.64 179.07 0)
 			(hide yes)
@@
 			)
 		)
-		(property "Footprint" "Capacitor_SMD:C_0402_1005Metric"
+		(property "Footprint" "pager-carrier:C_0402_1005Metric_NoSilk"
 			(at 199.39 62.23 0)
 			(hide yes)
@@
 			)
 		)
-		(property "Footprint" "Inductor_SMD:L_Murata_DFE201610P"
+		(property "Footprint" "pager-carrier:L_Murata_DFE201610P_NoSilk"
 			(at 256.54 45.72 0)
 			(hide yes)
@@
 			)
 		)
-		(property "Footprint" "Resistor_SMD:R_0402_1005Metric"
+		(property "Footprint" "pager-carrier:R_0402_1005Metric_NoSilk"
 			(at 64.77 50.8 0)
 			(hide yes)
@@
 			)
 		)
-		(property "Footprint" "Resistor_SMD:R_0402_1005Metric"
+		(property "Footprint" "pager-carrier:R_0402_1005Metric_NoSilk"
 			(at 146.05 59.69 0)
 			(hide yes)
@@
 			)
 		)
-		(property "Footprint" "Resistor_SMD:R_0402_1005Metric"
+		(property "Footprint" "pager-carrier:R_0402_1005Metric_NoSilk"
 			(at 215.9 50.8 0)
 			(hide yes)
@@
 			)
 		)
-		(property "Footprint" "Resistor_SMD:R_0402_1005Metric"
+		(property "Footprint" "pager-carrier:R_0402_1005Metric_NoSilk"
 			(at 19.05 134.62 0)
 			(hide yes)
@@
 			)
 		)
-		(property "Footprint" "Resistor_SMD:R_0402_1005Metric"
+		(property "Footprint" "pager-carrier:R_0402_1005Metric_NoSilk"
 			(at 71.12 113.03 0)
 			(hide yes)
@@
 			)
 		)
-		(property "Footprint" "Resistor_SMD:R_0402_1005Metric"
+		(property "Footprint" "pager-carrier:R_0402_1005Metric_NoSilk"
 			(at 36.83 129.54 0)
 			(hide yes)
@@
 			)
 		)
-		(property "Footprint" "Capacitor_SMD:C_0402_1005Metric"
+		(property "Footprint" "pager-carrier:C_0402_1005Metric_NoSilk"
 			(at 127 168.91 0)
 			(hide yes)

Commit message: BOM: move six passives to JLC basic parts, fix connector LCSC codes (no footprint changes)
Carrier: R32 2.2M -> 1M (C26083), C14 22nF -> 100nF (C1525), R1 22.1k -> 22k (C25768),
R2 47.5k -> 47k (C25792); J1 LCSC C160407 (SM08B), J2 MPN/LCSC SM04B-SRSS-TB C160404
to match its SH footprint.
Panel: C11 4.7uF under basic code C19666, D1-D3 NSR0530 -> B5819W (C8598, SOD-123 as
already on the board), R4 2.2R gets C22939.
Board footprint fields updated to match. ERC clean on both.

Co-Authored-By: Claude Fable 5.1 <noreply@anthropic.com>
Parts:
- C14: value 22nF -> 100nF; LCSC C337699 -> C1525; MPN CL05B223KB5NNNC -> CL05B104KO5NNNC
- R32: value 2.2M -> 1M; LCSC C11490 -> C26083; MPN 0402WGF2204TCE -> 0402WGF1004TCE
Changed lines of the file:
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@@
 			)
 		)
-		(property "Value" "22nF"
+		(property "Value" "100nF"
 			(at 70.104 121.412 0)
 			(show_name no)
@@
 			)
 		)
-		(property "MPN" "CL05B223KB5NNNC"
+		(property "MPN" "CL05B104KO5NNNC"
 			(at 77.47 135.89 0)
 			(hide yes)
@@
 			)
 		)
-		(property "LCSC" "C337699"
+		(property "LCSC" "C1525"
 			(at 77.47 138.43 0)
 			(hide yes)
@@
 			)
 		)
-		(property "Value" "2.2M"
+		(property "Value" "1M"
 			(at 85.344 121.666 0)
 			(show_name no)
@@
 			)
 		)
-		(property "MPN" "0402WGF2204TCE"
+		(property "MPN" "0402WGF1004TCE"
 			(at 83.82 135.89 0)
 			(hide yes)
@@
 			)
 		)
-		(property "LCSC" "C11490"
+		(property "LCSC" "C26083"
 			(at 83.82 138.43 0)
 			(hide yes)
