File: hardware/carrier/panel/panel_main.kicad_sch (KiCad schematic)
At the start: 28 parts, among them J1 GDEY029T94 FPC, J2 CARRIER, J3 FL-A FPC (FL03), J4 FL-B FPC (Orient), Q5 AO3400A

Commit message: Attempt to layout the PCB
Parts:
- C1: footprint Capacitor_SMD:C_0603_1608Metric -> Capacitor_SMD:C_0402_1005Metric; LCSC C19702 -> C15525; MPN CL10A106KP8NNNC -> CL05A106MQ5NUNC
- C11: value 4.7uF/25V -> 4.7uF; footprint Capacitor_SMD:C_0805_2012Metric -> Capacitor_SMD:C_0603_1608Metric; LCSC C1779 -> C1705; MPN CL21B475KAQNNNE -> CL10A475KP8NNNC
- C2, C6: footprint Capacitor_SMD:C_0603_1608Metric -> Capacitor_SMD:C_0402_1005Metric; LCSC C15849 -> C52923; MPN CL10A105KA8NNNC -> CL05A105KA5NQNC
- D1, D2, D3: value MBR0530 -> NSR0530; footprint Diode_SMD:D_SOD-123 -> Diode_SMD:D_SOD-323; LCSC C82046 -> C556393; MPN MBR0530 -> NSR0530HT1G
- L1: LCSC (none) -> C83435
- Q5: value AO3400A -> SI1308EDL; footprint Package_TO_SOT_SMD:SOT-23 -> Package_TO_SOT_SMD:SOT-323_SC-70; LCSC C20917 -> C469327; MPN AO3400A -> SI1308EDL-T1-GE3
- R1, R2, R3, R5: footprint Resistor_SMD:R_0603_1608Metric -> Resistor_SMD:R_0402_1005Metric; LCSC C21189 -> C17168; MPN 0603WAF0000T5E -> 0402WGF0000TCE
- R6, R7: footprint Resistor_SMD:R_0603_1608Metric -> Resistor_SMD:R_0402_1005Metric; LCSC C25804 -> C25744; MPN 0603WAF1002T5E -> 0402WGF1002TCE
- R8: footprint Resistor_SMD:R_0603_1608Metric -> Resistor_SMD:R_0402_1005Metric; LCSC C22935 -> C26083; MPN 0603WAF1004T5E -> 0402WGF1004TCE
Changed lines of the file:
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@@
 			)
 		)
-		(property "Value" "AO3400A"
+		(property "Value" "SI1308EDL"
 			(at 295.148 111.76 0)
 			(show_name no)
@@
 			)
 		)
-		(property "Footprint" "Package_TO_SOT_SMD:SOT-23"
+		(property "Footprint" "Package_TO_SOT_SMD:SOT-323_SC-70"
 			(at 293.37 110.49 0)
 			(hide yes)
@@
 			)
 		)
-		(property "Datasheet" "http://www.aosmd.com/pdfs/datasheet/AO3400A.pdf"
+		(property "Datasheet" "https://www.vishay.com/docs/73390/si1308edl.pdf"
 			(at 293.37 113.03 0)
 			(hide yes)
@@
 			)
 		)
-		(property "MPN" "AO3400A"
+		(property "MPN" "SI1308EDL-T1-GE3"
 			(at 289.56 125.73 0)
 			(hide yes)
@@
 			)
 		)
-		(property "LCSC" "C20917"
+		(property "LCSC" "C469327"
 			(at 289.56 128.27 0)
 			(hide yes)
@@
 			)
 		)
-		(property "Footprint" "Resistor_SMD:R_0603_1608Metric"
+		(property "Footprint" "Resistor_SMD:R_0402_1005Metric"
 			(at 222.25 217.17 0)
 			(hide yes)
@@
 			)
 		)
-		(property "MPN" "0603WAF0000T5E"
+		(property "MPN" "0402WGF0000TCE"
 			(at 220.98 231.14 0)
 			(hide yes)
@@
 			)
 		)
-		(property "LCSC" "C21189"
+		(property "LCSC" "C17168"
 			(at 220.98 233.68 0)
 			(hide yes)
@@
 			)
 		)
-		(property "Footprint" "Resistor_SMD:R_0603_1608Metric"
+		(property "Footprint" "Resistor_SMD:R_0402_1005Metric"
 			(at 280.67 128.27 0)
 			(hide yes)
@@
 			)
 		)
-		(property "MPN" "0603WAF1004T5E"
+		(property "MPN" "0402WGF1004TCE"
 			(at 279.4 142.24 0)
 			(hide yes)
@@
 			)
 		)
-		(property "LCSC" "C22935"
+		(property "LCSC" "C26083"
 			(at 279.4 144.78 0)
 			(hide yes)
@@
 			)
 		)
-		(property "Footprint" "Resistor_SMD:R_0603_1608Metric"
+		(property "Footprint" "Resistor_SMD:R_0402_1005Metric"
 			(at 184.15 217.17 0)
 			(hide yes)
@@
 			)
 		)
-		(property "MPN" "0603WAF0000T5E"
+		(property "MPN" "0402WGF0000TCE"
 			(at 182.88 231.14 0)
 			(hide yes)
@@
 			)
 		)
-		(property "LCSC" "C21189"
+		(property "LCSC" "C17168"
 			(at 182.88 233.68 0)
 			(hide yes)
@@
 			)
 		)
-		(property "Value" "MBR0530"
+		(property "Value" "NSR0530"
 			(at 246.38 116.078 0)
 			(show_name no)
@@
 			)
 		)
-		(property "Footprint" "Diode_SMD:D_SOD-123"
+		(property "Footprint" "Diode_SMD:D_SOD-323"
 			(at 240.03 123.19 0)
 			(hide yes)
@@
 			)
 		)
-		(property "MPN" "MBR0530"
+		(property "MPN" "NSR0530HT1G"
 			(at 245.11 134.62 0)
 			(hide yes)
@@
 			)
 		)
-		(property "LCSC" "C82046"
+		(property "LCSC" "C556393"
 			(at 245.11 137.16 0)
 			(hide yes)
@@
 			)
 		)
-		(property "Footprint" "Resistor_SMD:R_0603_1608Metric"
+		(property "Footprint" "Resistor_SMD:R_0402_1005Metric"
 			(at 196.85 217.17 0)
 			(hide yes)
@@
 			)
 		)
-		(property "MPN" "0603WAF0000T5E"
+		(property "MPN" "0402WGF0000TCE"
 			(at 195.58 231.14 0)
 			(hide yes)
@@
 			)
 		)
-		(property "LCSC" "C21189"
+		(property "LCSC" "C17168"
 			(at 195.58 233.68 0)
 			(hide yes)
@@
 			)
 		)
-		(property "LCSC" ""
+		(property "LCSC" "C83435"
 			(at 292.1 87.63 0)
 			(hide yes)
@@
 			)
 		)
-		(property "Footprint" "Resistor_SMD:R_0603_1608Metric"
+		(property "Footprint" "Resistor_SMD:R_0402_1005Metric"
 			(at 143.51 60.96 0)
 			(hide yes)
@@
 			)
 		)
-		(property "MPN" "0603WAF1002T5E"
+		(property "MPN" "0402WGF1002TCE"
 			(at 142.24 74.93 0)
 			(hide yes)
@@
 			)
 		)
-		(property "LCSC" "C25804"
+		(property "LCSC" "C25744"
 			(at 142.24 77.47 0)
 			(hide yes)
@@
 			)
 		)
-		(property "Footprint" "Capacitor_SMD:C_0603_1608Metric"
+		(property "Footprint" "Capacitor_SMD:C_0402_1005Metric"
 			(at 114.3 95.25 0)
 			(hide yes)
@@
 			)
 		)
-		(property "MPN" "CL10A105KA8NNNC"
+		(property "MPN" "CL05A105KA5NQNC"
 			(at 113.03 109.22 0)
 			(hide yes)
@@
 			)
 		)
-		(property "LCSC" "C15849"
+		(property "LCSC" "C52923"
 			(at 113.03 111.76 0)
 			(hide yes)
@@
 			)
 		)
-		(property "Footprint" "Capacitor_SMD:C_0603_1608Metric"
+		(property "Footprint" "Capacitor_SMD:C_0402_1005Metric"
 			(at 156.21 60.96 0)
 			(hide yes)
@@
 			)
 		)
-		(property "MPN" "CL10A106KP8NNNC"
+		(property "MPN" "CL05A106MQ5NUNC"
 			(at 154.94 74.93 0)
 			(hide yes)
@@
 			)
 		)
-		(property "LCSC" "C19702"
+		(property "LCSC" "C15525"
 			(at 154.94 77.47 0)
 			(hide yes)
@@
 			)
 		)
-		(property "Value" "MBR0530"
+		(property "Value" "NSR0530"
 			(at 243.586 130.302 0)
 			(show_name no)
@@
 			)
 		)
-		(property "Footprint" "Diode_SMD:D_SOD-123"
+		(property "Footprint" "Diode_SMD:D_SOD-323"
 			(at 250.19 129.54 0)
 			(hide yes)
@@
 			)
 		)
-		(property "MPN" "MBR0530"
+		(property "MPN" "NSR0530HT1G"
 			(at 245.11 140.97 0)
 			(hide yes)
@@
 			)
 		)
-		(property "LCSC" "C82046"
+		(property "LCSC" "C556393"
 			(at 245.11 143.51 0)
 			(hide yes)
@@
 			)
 		)
-		(property "Value" "4.7uF/25V"
+		(property "Value" "4.7uF"
 			(at 315.976 75.184 0)
 			(show_name no)
@@
 			)
 		)
-		(property "Footprint" "Capacitor_SMD:C_0805_2012Metric"
+		(property "Footprint" "Capacitor_SMD:C_0603_1608Metric"
 			(at 312.42 74.93 0)
 			(hide yes)
@@
 			)
 		)
-		(property "MPN" "CL21B475KAQNNNE"
+		(property "MPN" "CL10A475KP8NNNC"
 			(at 311.15 88.9 0)
 			(hide yes)
@@
 			)
 		)
-		(property "LCSC" "C1779"
+		(property "LCSC" "C1705"
 			(at 311.15 91.44 0)
 			(hide yes)
@@
 			)
 		)
-		(property "Footprint" "Capacitor_SMD:C_0603_1608Metric"
+		(property "Footprint" "Capacitor_SMD:C_0402_1005Metric"
 			(at 168.91 60.96 0)
 			(hide yes)
@@
 			)
 		)
-		(property "MPN" "CL10A105KA8NNNC"
+		(property "MPN" "CL05A105KA5NQNC"
 			(at 167.64 74.93 0)
 			(hide yes)
@@
 			)
 		)
-		(property "LCSC" "C15849"
+		(property "LCSC" "C52923"
 			(at 167.64 77.47 0)
 			(hide yes)
@@
 			)
 		)
-		(property "Footprint" "Resistor_SMD:R_0603_1608Metric"
+		(property "Footprint" "Resistor_SMD:R_0402_1005Metric"
 			(at 209.55 217.17 0)
 			(hide yes)
@@
 			)
 		)
-		(property "MPN" "0603WAF0000T5E"
+		(property "MPN" "0402WGF0000TCE"
 			(at 208.28 231.14 0)
 			(hide yes)
@@
 			)
 		)
-		(property "LCSC" "C21189"
+		(property "LCSC" "C17168"
 			(at 208.28 233.68 0)
 			(hide yes)
@@
 			)
 		)
-		(property "Footprint" "Resistor_SMD:R_0603_1608Metric"
+		(property "Footprint" "Resistor_SMD:R_0402_1005Metric"
 			(at 130.81 60.96 0)
 			(hide yes)
@@
 			)
 		)
-		(property "MPN" "0603WAF1002T5E"
+		(property "MPN" "0402WGF1002TCE"
 			(at 129.54 74.93 0)
 			(hide yes)
@@
 			)
 		)
-		(property "LCSC" "C25804"
+		(property "LCSC" "C25744"
 			(at 129.54 77.47 0)
 			(hide yes)
@@
 			)
 		)
-		(property "Value" "MBR0530"
+		(property "Value" "NSR0530"
 			(at 248.666 72.39 0)
 			(show_name no)
@@
 			)
 		)
-		(property "Footprint" "Diode_SMD:D_SOD-123"
+		(property "Footprint" "Diode_SMD:D_SOD-323"
 			(at 255.27 80.01 0)
 			(hide yes)
@@
 			)
 		)
-		(property "MPN" "MBR0530"
+		(property "MPN" "NSR0530HT1G"
 			(at 250.19 91.44 0)
 			(hide yes)
@@
 			)
 		)
-		(property "LCSC" "C82046"
+		(property "LCSC" "C556393"
 			(at 250.19 93.98 0)
 			(hide yes)
