File: hardware/carrier/panel/panel_main.kicad_sch (KiCad schematic)
At the start: 26 parts, among them J1 GDEY029T94 FPC, J2 CARRIER, J3 FL-A FPC (FL03), J5 FRONTLIGHT, Q5 SI1308EDL

Commit message: Panel: J1/J3 to SnapEDA FH34SRJ footprints (hold-downs at 2.5 mm, pin 1 per Hirose)
JLC flagged J1/J3: the custom footprints put the MP pads at y=3.3
(read the datasheet's 3.3 outer-edge span as centre-to-centre) and
had pin 1 mirrored.

Co-Authored-By: Claude Opus 5.5 <noreply@anthropic.com>
Parts:
- J1: value GDEY029T94 FPC -> FH34SRJ-24S-0.5SH_50_; footprint pager-carrier:Hirose_FH34SRJ-24S-0.5SH_1x24-1MP_P0.50mm_Horizontal -> h24:HRS_FH34SRJ-24S-0.5SH_50_; symbol Connector_Generic:Conn_01x24 -> FH34-26:FH34SRJ-24S-0.5SH_50_; Availability (none) -> In Stock; Check_prices (none) -> https://www.snapeda.com/parts/FH34SRJ-24S-0.5SH(50)/Hirose/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; MANUFACTURER (none) -> HRS; MF (none) -> Hirose Electric; MP (none) -> FH34SRJ-24S-0.5SH(50); Package (none) -> None; Price (none) -> None; SnapEDA_Link (none) -> https://www.snapeda.com/parts/FH34SRJ-24S-0.5SH(50)/Hirose/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
- J3: value FL-A FPC (FL03) -> FH34SRJ-6S-0.5SH_50_; footprint pager-carrier:Hirose_FH34SRJ-6S-0.5SH_1x06-1MP_P0.50mm_Horizontal -> h6:HRS_FH34SRJ-6S-0.5SH_50_; symbol Connector_Generic:Conn_01x06 -> FH34SRJ-6S-0.5SH(50):FH34SRJ-6S-0.5SH_50_; Availability (none) -> In Stock; Check_prices (none) -> https://www.snapeda.com/parts/FH34SRJ-6S-0.5SH(50)/Hirose+E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; MANUFACTURER (none) -> HRS; MF (none) -> Hirose Electric Co Ltd; MP (none) -> FH34SRJ-6S-0.5SH(50); Package (none) -> None; Price (none) -> None; SnapEDA_Link (none) -> https://www.snapeda.com/parts/FH34SRJ-6S-0.5SH(50)/Hirose+E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
Connections:
- net GND: now also J1.S1 (SHIELD), J1.S2 (SHIELD), J3.S1 (SHIELD), J3.S2 (SHIELD)
- no-connect marks 7 -> 8
Other:
- moved on the sheet: J5, JP1, JP2
