File: hardware/carrier/panel/pager-panel.kicad_pcb (KiCad board)
At the start: 2 copper layers, 32 x 20 mm, 26 parts, among them J1 GDEY029T94 FPC, J2 CARRIER, J3 FL-A FPC (FL03), J5 FRONTLIGHT, Q5 SI1308EDL

Commit message: Finalizing PCB cute designs
Routing:
- net (no net): track 0.00 -> 22.5 mm
Other:
- board text added: "Oct '26 @awongawong"
- board text removed: "@awongawong"
